Commit message: Serial comm + ros2_control + whole motor control &&  All PWM and PID are on Arduino

File: my_ws/src/my_robot_description/urdf/lidar.xacro (robot description, xacro)
@@ -19,5 +19,5 @@
           <min>0.10</min>
           <max>20.0</max>
-          <resolution>0.01</resolution>
+          <resolution>0.05</resolution>
         </range>
       </ray>

File: my_ws/src/my_robot_description/urdf/mobile_base.xacro (robot description, xacro)
@@ -9,4 +9,9 @@
     <xacro:property name="wheel_length" value="0.05" />
     <link name="base_footprint" />
+    <joint name ="base_joint" type="fixed">
+        <parent link="base_footprint" />
+        <child link="base_link" />
+        <origin xyz="0 0 ${wheel_radius}" rpy="0 0 0" />
+    </joint>
     <link name ="base_link">
         <visual>
@@ -91,9 +96,4 @@
     </link>
     <!--link relationship ==> joint-->
-    <joint name ="base_joint" type="fixed">
-        <parent link="base_footprint" />
-        <child link="base_link" />
-        <origin xyz="0 0 ${wheel_radius}" rpy="0 0 0" />
-    </joint>
     <joint name="base_lidar_joint" type="fixed">
         <parent link="base_link" />

File: my_ws/src/my_robot_description/urdf/my_robot_main.urdf.xacro (robot description, xacro)
@@ -8,4 +8,5 @@
     <xacro:include filename="mobile_base.xacro" />
     <xacro:include filename="mobile_base_gazebo.xacro" />
+    <xacro:include filename="ros2_control.xacro" />
     <!--rbotic arm -->
     <!-- <xacro:include filename="arm.xacro" />
